Commit message: simulation.launch

File: kuka_lwr/lwr_description/model/kuka_lwr.urdf.xacro (robot description, xacro)
@@ -332,3 +332,7 @@
     <xacro:kuka_lwr_transmission name="${name}"/>
   </xacro:macro>
+    <!-- using the models -->
+    <xacro:kuka_lwr name="lwr">
+        <origin xyz="0 0 0" rpy="0 0 0"/>
+    </xacro:kuka_lwr>
 </robot>
